File: kicad/GW1NR.kicad_sch (KiCad schematic)
At the start: 42 parts, among them U4 74LCX16245, U5 74LCX16245, U6 GW1NR-4&4B_QN881, U7 74LCX16245, U8 74LS06, U9 74LS06

Commit message: started routing
Connections:
- net D0_t: now also U6.77 (IOT30B); no longer U6.75 (IOT32B)
- net D1_t: now also U6.76 (IOT31B); no longer U6.74 (IOT33B)
- net D2_t: now also U6.75 (IOT32B); no longer U6.73 (IOT35A)
- net D3_t: now also U6.74 (IOT33B); no longer U6.72 (IOT35B)
- net D4_t: now also U6.73 (IOT35A); no longer U6.71 (IOT36A)
- net D5_t: now also U6.72 (IOT35B); no longer U6.70 (IOT36B)
- net D6_t: now also U6.71 (IOT36A); no longer U6.69 (IOT37A)
- net D7_t: now also U6.70 (IOT36B); no longer U6.68 (IOT37B)
- net ~{ROMH_t}: now also U6.69 (IOT37A); no longer U6.76 (IOT31B)
- net ~{ROML_t}: now also U6.68 (IOT37B); no longer U6.77 (IOT30B)
Changed lines of the file:
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@@
     (stroke (width 0) (type default) (color 0 0 0 0))
   )
+  (wire (pts (xy 273.05 74.93) (xy 274.32 74.93))
+    (stroke (width 0) (type default) (color 0 0 0 0))
+  )
   (wire (pts (xy 204.47 73.66) (xy 207.01 73.66))
     (stroke (width 0) (type default) (color 0 0 0 0))
   )
+  (wire (pts (xy 273.05 57.15) (xy 274.32 57.15))
+    (stroke (width 0) (type default) (color 0 0 0 0))
+  )
   (wire (pts (xy 69.85 31.75) (xy 69.85 36.83))
     (stroke (width 0) (type default) (color 0 0 0 0))
@@
     (stroke (width 0) (type default) (color 0 0 0 0))
   )
+  (wire (pts (xy 273.05 83.82) (xy 274.32 83.82))
+    (stroke (width 0) (type default) (color 0 0 0 0))
+  )
   (wire (pts (xy 157.48 163.83) (xy 161.29 163.83))
     (stroke (width 0) (type default) (color 0 0 0 0))
@@
     (stroke (width 0) (type default) (color 0 0 0 0))
   )
+  (wire (pts (xy 273.05 66.04) (xy 274.32 66.04))
+    (stroke (width 0) (type default) (color 0 0 0 0))
+  )
   (wire (pts (xy 57.15 138.43) (xy 59.69 138.43))
     (stroke (width 0) (type default) (color 0 0 0 0))
@@
     (effects (font (size 1.27 1.27)) (justify right bottom))
   )
-  (label "D7_t" (at 218.44 153.67 180)
+  (label "D7_t" (at 218.44 148.59 180)
     (effects (font (size 1.27 1.27)) (justify right bottom))
   )
@@
     (effects (font (size 1.27 1.27)) (justify right bottom))
   )
-  (label "D6_t" (at 218.44 151.13 180)
+  (label "D6_t" (at 218.44 146.05 180)
     (effects (font (size 1.27 1.27)) (justify right bottom))
   )
@@
     (effects (font (size 1.27 1.27)) (justify right bottom))
   )
-  (label "D0_t" (at 218.44 135.89 180)
+  (label "D0_t" (at 218.44 130.81 180)
     (effects (font (size 1.27 1.27)) (justify right bottom))
   )
@@
     (effects (font (size 1.27 1.27)) (justify left bottom))
   )
-  (label "~{ROMH_t}" (at 218.44 133.35 180)
+  (label "~{ROMH_t}" (at 218.44 151.13 180)
     (effects (font (size 1.27 1.27)) (justify right bottom))
   )
@@
     (effects (font (size 1.27 1.27)) (justify left bottom))
   )
-  (label "~{ROML_t}" (at 218.44 130.81 180)
+  (label "~{ROML_t}" (at 218.44 153.67 180)
     (effects (font (size 1.27 1.27)) (justify right bottom))
   )
@@
     (effects (font (size 1.27 1.27)) (justify right bottom))
   )
-  (label "D3_t" (at 218.44 143.51 180)
+  (label "D3_t" (at 218.44 138.43 180)
     (effects (font (size 1.27 1.27)) (justify right bottom))
   )
@@
     (effects (font (size 1.27 1.27)) (justify right bottom))
   )
-  (label "D2_t" (at 218.44 140.97 180)
+  (label "D2_t" (at 218.44 135.89 180)
     (effects (font (size 1.27 1.27)) (justify right bottom))
   )
@@
     (effects (font (size 1.27 1.27)) (justify right bottom))
   )
-  (label "D4_t" (at 218.44 146.05 180)
+  (label "D4_t" (at 218.44 140.97 180)
     (effects (font (size 1.27 1.27)) (justify right bottom))
   )
@@
     (effects (font (size 1.27 1.27)) (justify right bottom))
   )
-  (label "D1_t" (at 218.44 138.43 180)
+  (label "D1_t" (at 218.44 133.35 180)
     (effects (font (size 1.27 1.27)) (justify right bottom))
   )
-  (label "D5_t" (at 218.44 148.59 180)
+  (label "D5_t" (at 218.44 143.51 180)
     (effects (font (size 1.27 1.27)) (justify right bottom))
   )
@@
     (effects (font (size 1.27 1.27)) (justify left))
   )
-  (hierarchical_label "IEC_SRQ" (shape input) (at 273.05 83.82 0)
+  (hierarchical_label "IEC_SRQ" (shape input) (at 274.32 83.82 0)
     (effects (font (size 1.27 1.27)) (justify left))
   )
-  (hierarchical_label "IEC_CLK" (shape input) (at 273.05 66.04 0)
+  (hierarchical_label "IEC_CLK" (shape input) (at 274.32 66.04 0)
     (effects (font (size 1.27 1.27)) (justify left))
   )
@@
     (effects (font (size 1.27 1.27)) (justify right))
   )
-  (hierarchical_label "IEC_ATN" (shape input) (at 273.05 74.93 0)
+  (hierarchical_label "IEC_ATN" (shape input) (at 274.32 74.93 0)
     (effects (font (size 1.27 1.27)) (justify left))
   )
@@
     (effects (font (size 1.27 1.27)) (justify right))
   )
-  (hierarchical_label "IEC_DAT" (shape input) (at 273.05 57.15 0)
+  (hierarchical_label "IEC_DAT" (shape input) (at 274.32 57.15 0)
     (effects (font (size 1.27 1.27)) (justify left))
   )
@@
     (in_bom yes) (on_board yes)
     (property "Reference" "U8" (id 0) (at 264.16 66.04 0))
-    (property "Value" "74LS06" (id 1) (at 270.51 68.58 0))
+    (property "Value" "74LS06" (id 1) (at 267.97 69.85 0))
     (property "Footprint" "Package_SO:SO-14_3.9x8.65mm_P1.27mm" (id 2) (at 265.43 66.04 0)
       (effects (font (size 1.27 1.27)) hide)
@@
     (in_bom yes) (on_board yes)
     (property "Reference" "U8" (id 0) (at 264.16 83.82 0))
-    (property "Value" "74LS06" (id 1) (at 270.51 86.36 0))
+    (property "Value" "74LS06" (id 1) (at 269.24 87.63 0))
     (property "Footprint" "Package_SO:SO-14_3.9x8.65mm_P1.27mm" (id 2) (at 265.43 83.82 0)
       (effects (font (size 1.27 1.27)) hide)
@@
     (in_bom yes) (on_board yes)
     (property "Reference" "U8" (id 0) (at 264.16 74.93 0))
-    (property "Value" "74LS06" (id 1) (at 270.51 77.47 0))
+    (property "Value" "74LS06" (id 1) (at 269.24 78.74 0))
     (property "Footprint" "Package_SO:SO-14_3.9x8.65mm_P1.27mm" (id 2) (at 265.43 74.93 0)
       (effects (font (size 1.27 1.27)) hide)
@@
     (in_bom yes) (on_board yes)
     (property "Reference" "U8" (id 0) (at 264.16 57.15 0))
-    (property "Value" "74LS06" (id 1) (at 270.51 59.69 0))
+    (property "Value" "74LS06" (id 1) (at 267.97 60.96 0))
     (property "Footprint" "Package_SO:SO-14_3.9x8.65mm_P1.27mm" (id 2) (at 265.43 57.15 0)
       (effects (font (size 1.27 1.27)) hide)

Commit message: footprint fixed and gerber files, as ordered at JLCPCB
Parts:
- U4, U5, U7: footprint SOP50:SOP50P810X120-48N -> Package_SO:SSOP-48_5.3x12.8mm_P0.5mm
Changed lines of the file:
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@@
     (property "Reference" "U4" (id 0) (at 45.72 105.41 0))
     (property "Value" "74LCX16245" (id 1) (at 45.72 107.95 0))
-    (property "Footprint" "SOP50:SOP50P810X120-48N" (id 2) (at 45.72 146.05 0)
+    (property "Footprint" "Package_SO:SSOP-48_5.3x12.8mm_P0.5mm" (id 2) (at 45.72 146.05 0)
       (effects (font (size 1.27 1.27)) (justify left bottom) hide)
     )
@@
     (property "Reference" "U5" (id 0) (at 96.52 105.41 0))
     (property "Value" "74LCX16245" (id 1) (at 96.52 107.95 0))
-    (property "Footprint" "SOP50:SOP50P810X120-48N" (id 2) (at 96.52 146.05 0)
+    (property "Footprint" "Package_SO:SSOP-48_5.3x12.8mm_P0.5mm" (id 2) (at 96.52 146.05 0)
       (effects (font (size 1.27 1.27)) (justify left bottom) hide)
     )
@@
     (property "Reference" "U7" (id 0) (at 146.05 105.41 0))
     (property "Value" "74LCX16245" (id 1) (at 146.05 107.95 0))
-    (property "Footprint" "SOP50:SOP50P810X120-48N" (id 2) (at 146.05 146.05 0)
+    (property "Footprint" "Package_SO:SSOP-48_5.3x12.8mm_P0.5mm" (id 2) (at 146.05 146.05 0)
       (effects (font (size 1.27 1.27)) (justify left bottom) hide)
     )
